Commit message: Implement code to have the robot follow the track

File: urdf/robot.xacro (robot description, xacro)
@@ -141,7 +141,49 @@
     <material>Gazebo/Orange</material>
   </gazebo>
+  <!--
   <gazebo reference="camera_link">
     <material>Gazebo/Blue</material>
   </gazebo>
+  -->
+  <gazebo reference="camera_link">
+    <material>Gazebo/Blue</material>
+    <sensor type="camera" name="camera1">
+      <update_rate>30.0</update_rate>
+      <camera name="head">
+        <horizontal_fov>1.3962634</horizontal_fov>
+        <image>
+          <width>800</width>
+          <height>800</height>
+          <format>R8G8B8</format>
+        </image>
+        <clip>
+          <near>0.02</near>
+          <far>300</far>
+        </clip>
+        <noise>
+          <type>gaussian</type>
+          <!-- Noise is sampled independently per pixel on each frame.
+               That pixel's noise value is added to each of its color
+               channels, which at that point lie in the range [0,1]. -->
+          <mean>0.0</mean>
+          <stddev>0.007</stddev>
+        </noise>
+      </camera>
+      <plugin name="camera_controller" filename="libgazebo_ros_camera.so">
+        <alwaysOn>true</alwaysOn>
+        <updateRate>0.0</updateRate>
+        <cameraName>robot/camera</cameraName>
+        <imageTopicName>image_raw</imageTopicName>
+        <cameraInfoTopicName>camera_info</cameraInfoTopicName>
+        <frameName>camera_link</frameName>
+        <hackBaseline>0.07</hackBaseline>
+        <distortionK1>0.0</distortionK1>
+        <distortionK2>0.0</distortionK2>
+        <distortionK3>0.0</distortionK3>
+        <distortionT1>0.0</distortionT1>
+        <distortionT2>0.0</distortionT2>
+      </plugin>
+    </sensor>
+  </gazebo>
   <gazebo reference="wheel_FL">
     <material>Gazebo/Yellow</material>
@@ -156,3 +198,19 @@
     <material>Gazebo/Yellow</material>
   </gazebo>
+  <gazebo>
+  <plugin name="skid_steer_drive_controller" filename="libgazebo_ros_skid_steer_drive.so">
+    <updateRate>100.0</updateRate>
+    <robotNamespace>/</robotNamespace>
+    <leftFrontJoint>wheel_FL_joint</leftFrontJoint>
+    <rightFrontJoint>wheel_FR_joint</rightFrontJoint>
+    <leftRearJoint>wheel_RL_joint</leftRearJoint>
+    <rightRearJoint>wheel_RR_joint</rightRearJoint>
+    <wheelSeparation>2*${chassis_length/2-wheel_radius}</wheelSeparation>
+    <wheelDiameter>2*${wheel_radius}</wheelDiameter>
+    <robotBaseFrame>chassis</robotBaseFrame>
+    <torque>20</torque>
+    <topicName>cmd_vel</topicName>
+    <broadcastTF>false</broadcastTF>
+  </plugin>
+</gazebo>
 </robot>
